File: PCB/ESP Breakout/ESP_Breakout.sch (KiCad schematic (older format))
At the start: 3 parts, among them J1 Conn_01x11_Male, J2 Conn_01x11_Male, U1 ESP-12E

Commit message: new code
Connections:
- net at U1.1 (REST): no longer J1.1 (Pin_1)
- net at U1.10 (GPIO15): no longer J2.5 (Pin_5)
- net at U1.11 (GPIO2): no longer J2.6 (Pin_6)
- net at U1.12 (GPIO0): no longer J2.7 (Pin_7)
- net at U1.13 (GPIO4): no longer J2.8 (Pin_8)
- net at U1.14 (GPIO5): no longer J2.9 (Pin_9)
- net at U1.15 (RXD): no longer J2.10 (Pin_10)
- net at U1.16 (TXD): no longer J2.11 (Pin_11)
- net at U1.17 (CS0): no longer J1.9 (Pin_9)
- net at U1.18 (MISO): no longer J1.10 (Pin_10)
- net at U1.19 (GPIO9): no longer J1.11 (Pin_11)
- net at U1.2 (ADC): no longer J1.2 (Pin_2)
- net at U1.20 (GPIO10): no longer J2.1 (Pin_1)
- net at U1.21 (MOSI): no longer J2.2 (Pin_2)
- net at U1.22 (SCLK): no longer J2.3 (Pin_3)
- net at U1.3 (CH_PD): no longer J1.3 (Pin_3)
- net at U1.4 (GPIO16): no longer J1.4 (Pin_4)
- net at U1.5 (GPIO14): no longer J1.5 (Pin_5)
- net at U1.6 (GPIO12): no longer J1.6 (Pin_6)
- net at U1.7 (GPIO13): no longer J1.7 (Pin_7)
- net at U1.8 (VCC): no longer J1.8 (Pin_8)
- net at U1.9 (GND): no longer J2.4 (Pin_4)
Changed lines of the file:
@@
 EESchema Schematic File Version 2
-LIBS:ESP8266
 LIBS:power
 LIBS:device
@@
 LIBS:contrib
 LIBS:valves
+LIBS:ESP8266
 LIBS:ESP_Breakout-cache
 EELAYER 25 0
@@
 $Comp
 L ESP-12E U1
-U 1 1 5BD496BF
-P 5350 3250
-F 0 "U1" H 5350 3150 50  0000 C CNN
-F 1 "ESP-12E" H 5350 3350 50  0000 C CNN
-F 2 "ESP8266:ESP-12E_SMD" H 5350 3250 50  0001 C CNN
-F 3 "" H 5350 3250 50  0001 C CNN
-	1    5350 3250
+U 1 1 5BFEEA46
+P 5000 5850
+F 0 "U1" H 5000 5750 50  0000 C CNN
+F 1 "ESP-12E" H 5000 5950 50  0000 C CNN
+F 2 "ESP8266:ESP-12E_SMD" H 5000 5850 50  0001 C CNN
+F 3 "" H 5000 5850 50  0001 C CNN
+	1    5000 5850
 	1    0    0    -1
 $EndComp
 $Comp
 L Conn_01x11_Male J2
-U 1 1 5BD4A960
-P 7150 3350
-F 0 "J2" H 7150 3950 50  0000 C CNN
-F 1 "Conn_01x11_Male" H 7150 2750 50  0000 C CNN
-F 2 "Pin_Headers:Pin_Header_Straight_1x11_Pitch2.54mm" H 7150 3350 50  0001 C CNN
-F 3 "" H 7150 3350 50  0001 C CNN
-	1    7150 3350
-	-1   0    0    1
+U 1 1 5BFEEAA5
+P 6550 6000
+F 0 "J2" H 6550 6600 50  0000 C CNN
+F 1 "Conn_01x11_Male" H 6550 5400 50  0000 C CNN
+F 2 "Pin_Headers:Pin_Header_Straight_1x11_Pitch2.54mm" H 6550 6000 50  0001 C CNN
+F 3 "" H 6550 6000 50  0001 C CNN
+	1    6550 6000
+	1    0    0    -1
 $EndComp
 $Comp
 L Conn_01x11_Male J1
-U 1 1 5BD4A99D
-P 3550 3350
-F 0 "J1" H 3550 3950 50  0000 C CNN
-F 1 "Conn_01x11_Male" H 3550 2750 50  0000 C CNN
-F 2 "Pin_Headers:Pin_Header_Straight_1x11_Pitch2.54mm" H 3550 3350 50  0001 C CNN
-F 3 "" H 3550 3350 50  0001 C CNN
-	1    3550 3350
+U 1 1 5BFEEAE9
+P 3400 5900
+F 0 "J1" H 3400 6500 50  0000 C CNN
+F 1 "Conn_01x11_Male" H 3400 5300 50  0000 C CNN
+F 2 "Pin_Headers:Pin_Header_Straight_1x11_Pitch2.54mm" H 3400 5900 50  0001 C CNN
+F 3 "" H 3400 5900 50  0001 C CNN
+	1    3400 5900
 	1    0    0    -1
 $EndComp
-Wire Wire Line
-	3750 2850 4450 2950
-Wire Wire Line
-	3750 2950 4450 3050
-Wire Wire Line
-	3750 3050 4450 3150
-Wire Wire Line
-	3750 3150 4450 3250
-Wire Wire Line
-	3750 3250 4450 3350
-Wire Wire Line
-	3750 3350 4450 3450
-Wire Wire Line
-	3750 3450 4450 3550
-Wire Wire Line
-	3750 3550 4450 3650
-Wire Wire Line
-	5100 4150 3750 3650
-Wire Wire Line
-	3750 3750 5200 4150
-Wire Wire Line
-	5300 4150 3750 3850
-Wire Wire Line
-	6250 2950 6950 2850
-Wire Wire Line
-	6250 3050 6950 2950
-Wire Wire Line
-	6250 3150 6950 3050
-Wire Wire Line
-	6250 3250 6950 3150
-Wire Wire Line
-	6250 3350 6950 3250
-Wire Wire Line
-	6250 3450 6950 3350
-Wire Wire Line
-	6250 3550 6950 3450
-Wire Wire Line
-	6250 3650 6950 3550
-Wire Wire Line
-	6950 3650 5600 4150
-Wire Wire Line
-	6950 3750 5500 4150
-Wire Wire Line
-	6950 3850 5400 4150
 $EndSCHEMATC
